File: copyHHKB.kicad_pcb (KiCad board)
At the start: 2 copper layers, 121 parts, among them U1 ARDUINO_MICRO_SHIELD, j1 SW_DIP_x01, k1 SW_DIP_x01, m1 SW_DIP_x01, p1 SW_DIP_x01, q1 SW_DIP_x01, t1 SW_DIP_x01, u1 SW_DIP_x01, x1 SW_DIP_x01, y1 SW_DIP_x01

Commit message: 割と実際のサイズを計算してスイッチを着始めた
0.05mm大きいけど気にしない方向性
Parts:
- moved U1 123.0 mm to (282.7, 116.1)
- moved D49 121.4 mm to (-8.13, 151.6)
- moved AltL1 121.3 mm to (0.76, 147.8)
- moved D50 112.7 mm to (20.3, 151.6)
- moved winL1 112.7 mm to (29.0, 147.8)
- moved D52 94.1 mm to (153.4, 151.6)
- moved winR1 93.2 mm to (162.6, 147.3)
- moved D51 87.2 mm to (86.4, 151.6)
- moved SP1 86.3 mm to (95.5, 147.8)
- moved D53 85.9 mm to (182.4, 151.6)
- moved D4 85.0 mm to (-13.2, 132.6)
- moved AltR1 84.9 mm to (191.3, 147.8)
- moved shiftL1 84.2 mm to (-4.32, 128.8)
- moved D3 84.0 mm to (-18.3, 113.5)
- moved Control1 84.0 mm to (-9.40, 109.7)
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Routing:
- net (no net): track 0.00 -> 102.0 mm

Commit message: とりあえず動くレベル
Parts:
- added G***: LOGO, logo:HHKBlogo, F.Cu at (259.1, 125.7)
- added G***: LOGO, logo:free, F.Cu at (184.2, 90.2)
- added G***: LOGO, logo:megane, F.Cu at (63.5, 88.9)
- added REF**: MountingHole_3.2mm_M3_DIN965, Mounting_Holes:MountingHole_3.2mm_M3_DIN965, F.Cu at (195.6, 58.4)
- added REF**: MountingHole_3.2mm_M3_DIN965, Mounting_Holes:MountingHole_3.2mm_M3_DIN965, F.Cu at (241.3, 87.6)
- added REF**: MountingHole_3.2mm_M3_DIN965, Mounting_Holes:MountingHole_3.2mm_M3_DIN965, F.Cu at (274.3, 87.6)
- added REF**: MountingHole_3.2mm_M3_DIN965, Mounting_Holes:MountingHole_3.2mm_M3_DIN965, F.Cu at (184.2, 129.5)
- added REF**: MountingHole_3.2mm_M3_DIN965, Mounting_Holes:MountingHole_3.2mm_M3_DIN965, F.Cu at (139.7, 120.7)
- added REF**: MountingHole_3.2mm_M3_DIN965, Mounting_Holes:MountingHole_3.2mm_M3_DIN965, F.Cu at (114.3, 119.4)
- added REF**: MountingHole_3.2mm_M3_DIN965, Mounting_Holes:MountingHole_3.2mm_M3_DIN965, F.Cu at (19.1, 120.7)
- added REF**: MountingHole_3.2mm_M3_DIN965, Mounting_Holes:MountingHole_3.2mm_M3_DIN965, F.Cu at (80.8, 58.9)
- added REF**: MountingHole_3.2mm_M3_DIN965, Mounting_Holes:MountingHole_3.2mm_M3_DIN965, F.Cu at (209.8, 97.5)
- added REF**: MountingHole_3.2mm_M3_DIN965, Mounting_Holes:MountingHole_3.2mm_M3_DIN965, F.Cu at (77.2, 97.0)
- added REF**: MountingHole_3.2mm_M3_DIN965, Mounting_Holes:MountingHole_3.2mm_M3_DIN965, F.Cu at (48.3, 77.5)
- added REF**: MountingHole_3.2mm_M3_DIN965, Mounting_Holes:MountingHole_3.2mm_M3_DIN965, F.Cu at (181.6, 77.5)
- added REF**: MountingHole_3.2mm_M3_DIN965, Mounting_Holes:MountingHole_3.2mm_M3_DIN965, F.Cu at (105.4, 77.5)
- added REF**: MountingHole_3.2mm_M3_DIN965, Mounting_Holes:MountingHole_3.2mm_M3_DIN965, F.Cu at (25.4, 82.5)
- added REF**: MountingHole_3.2mm_M3_DIN965, Mounting_Holes:MountingHole_3.2mm_M3_DIN965, F.Cu at (255.3, 62.2)
- U1: moved to B.Cu
- moved U1 176.7 mm to (110.0, 78.6), turned to 0 degrees
- moved D52 42.1 mm to (189.2, 129.5)
- moved winR1 41.6 mm to (198.1, 125.7)
- moved D49 39.5 mm to (24.6, 129.5)
- moved AltL1 39.5 mm to (33.5, 125.7)
- moved D51 38.7 mm to (118.1, 129.5)
- moved SP1 38.5 mm to (127.0, 125.7)
- moved D53 37.0 mm to (212.1, 129.5)
- moved AltR1 37.0 mm to (221.0, 125.7)
- moved winL1 35.2 mm to (56.4, 125.7)
- moved D50 35.0 mm to (47.5, 129.5)
- moved D54 34.7 mm to (237.5, 109.7)
- moved shiftR1 34.4 mm to (245.9, 105.9)
- moved &1 33.2 mm to (139.2, 48.8)
- moved )1 33.2 mm to (196.3, 48.8)
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Routing:
- net row4: track 0.00 -> 415.1 mm, vias 0 -> 3
- net col9: track 0.00 -> 294.2 mm, vias 0 -> 4
- net row3: track 0.00 -> 288.9 mm
- net row0: track 0.00 -> 283.1 mm
- net row1: track 0.00 -> 272.1 mm
- net row2: track 0.00 -> 261.5 mm
- net col13: track 0.00 -> 226.6 mm, vias 0 -> 2
- net col1: track 0.00 -> 188.3 mm, vias 0 -> 3
- net col0: track 0.00 -> 187.7 mm
- net col2: track 0.00 -> 184.5 mm, vias 0 -> 9
- net col11: track 0.00 -> 178.6 mm, vias 0 -> 4
- net col12: track 0.00 -> 164.2 mm, vias 0 -> 3
- net col10: track 0.00 -> 153.3 mm, vias 0 -> 2
- net col3: track 0.00 -> 148.3 mm, vias 0 -> 6
- net col5: track 0.00 -> 143.0 mm, vias 0 -> 1
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Other:
- board outline added: 289.6 x 96.5 mm
- board text added: "@bamboorobo5884"

Commit message: 色々問題発覚したのでそれの修正
microのPINとスイッチが干渉してたので
microの位置を右下に変更
Parts:
- removed the G*** at (184.2, 90.2)
- removed the REF** at (195.6, 58.4)
- removed the REF** at (241.3, 87.6)
- removed the REF** at (274.3, 87.6)
- removed the REF** at (184.2, 129.5)
- removed the REF** at (139.7, 120.7)
- removed the REF** at (114.3, 119.4)
- removed the REF** at (19.1, 120.7)
- removed the REF** at (80.8, 58.9)
- removed the REF** at (209.8, 97.5)
- removed the REF** at (77.2, 97.0)
- removed the REF** at (48.3, 77.5)
- removed the REF** at (181.6, 77.5)
- removed the REF** at (105.4, 77.5)
- removed the REF** at (25.4, 82.5)
- removed the REF** at (255.3, 62.2)
- added G***: LOGO, logo:HHKBlogo, B.Cu at (256.5, 125.7)
- added G***: LOGO, logo:megane, B.Cu at (199.4, 83.8)
- added REF**: MountingHole_3.2mm_M3, Mounting_Holes:MountingHole_3.2mm_M3, F.Cu at (181.4, 77.7)
- added REF**: MountingHole_3.2mm_M3, Mounting_Holes:MountingHole_3.2mm_M3, F.Cu at (105.4, 124.5)
- added REF**: MountingHole_3.2mm_M3, Mounting_Holes:MountingHole_3.2mm_M3, F.Cu at (146.1, 123.2)
- added REF**: MountingHole_3.2mm_M3, Mounting_Holes:MountingHole_3.2mm_M3, F.Cu at (274.3, 87.6)
- added REF**: MountingHole_3.2mm_M3, Mounting_Holes:MountingHole_3.2mm_M3, F.Cu at (246.9, 82.8)
- added REF**: MountingHole_3.2mm_M3, Mounting_Holes:MountingHole_3.2mm_M3, F.Cu at (86.3, 77.6)
- added REF**: MountingHole_3.2mm_M3, Mounting_Holes:MountingHole_3.2mm_M3, F.Cu at (195.6, 58.9)
- added REF**: MountingHole_3.2mm_M3, Mounting_Holes:MountingHole_3.2mm_M3, F.Cu at (99.9, 58.5)
- added REF**: MountingHole_3.2mm_M3, Mounting_Holes:MountingHole_3.2mm_M3, F.Cu at (95.8, 96.9)
- added REF**: MountingHole_3.2mm_M3, Mounting_Holes:MountingHole_3.2mm_M3, F.Cu at (172.2, 97.2)
- added REF**: MountingHole_3.2mm_M3, Mounting_Holes:MountingHole_3.2mm_M3, F.Cu at (279.4, 61.0)
- added REF**: MountingHole_3.2mm_M3, Mounting_Holes:MountingHole_3.2mm_M3, F.Cu at (-2.54, 62.2)
- added REF**: MountingHole_3.2mm_M3, Mounting_Holes:MountingHole_3.2mm_M3, F.Cu at (2.54, 128.3)
- moved U1 179.6 mm to (280.7, 134.5), turned to 180 degrees
- moved G*** 25.9 mm to (88.9, 83.8)
Routing:
- net col6: track 69.7 -> 207.7 mm
- net col7: track 69.3 -> 202.6 mm
- net col4: track 115.1 -> 243.3 mm, vias 3 -> 0
- net col13: track 226.6 -> 102.0 mm, vias 2 -> 0
- net col0: track 187.7 -> 304.6 mm
- net col1: track 188.3 -> 302.2 mm, vias 3 -> 1
- net col2: track 184.5 -> 285.1 mm, vias 9 -> 0
- net row0: track 283.1 -> 376.4 mm
- net col3: track 148.3 -> 238.5 mm, vias 6 -> 1
- net row1: track 272.1 -> 346.4 mm, vias 0 -> 2
- net col5: track 143.0 -> 213.3 mm
- net col8: track 121.7 -> 187.4 mm, vias 4 -> 0
- net row4: track 415.1 -> 352.5 mm, vias 3 -> 1
- net col11: track 178.6 -> 122.5 mm, vias 4 -> 1
- net col12: track 164.2 -> 123.9 mm, vias 3 -> 2
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- added copper zone on B.Cu, net Net-(U1-PadGND)
- added copper zone on F.Cu, net Net-(U1-PadGND)
