File: copyHHKB2.kicad_pcb (KiCad board)
At the start: 2 copper layers, 289.6 x 96.5 mm, 124 parts, among them U1 ARDUINO_MICRO_SHIELD, j1 SW_DIP_x01, k1 SW_DIP_x01, m1 SW_DIP_x01, p1 SW_DIP_x01, q1 SW_DIP_x01, t1 SW_DIP_x01, u1 SW_DIP_x01, x1 SW_DIP_x01, y1 SW_DIP_x01

Commit message: logoとか追加
Parts:
- removed the G*** at (259.1, 125.7)
- added G***: LOGO, logo:HHKBlogo, B.Cu at (254.3, 127.0)
- added G***: LOGO, logo:HHKBlogo, F.Cu at (255.3, 127.0)
- added REF**: MountingHole_3.2mm_M3, Mounting_Holes:MountingHole_3.2mm_M3, F.Cu at (279.4, 62.5)
- added REF**: MountingHole_3.2mm_M3, Mounting_Holes:MountingHole_3.2mm_M3, F.Cu at (105.1, 78.2)
- added REF**: MountingHole_3.2mm_M3, Mounting_Holes:MountingHole_3.2mm_M3, F.Cu at (-2.29, 61.7)
- added REF**: MountingHole_3.2mm_M3, Mounting_Holes:MountingHole_3.2mm_M3, F.Cu at (0.05, 123.2)
- added REF**: MountingHole_3.2mm_M3, Mounting_Holes:MountingHole_3.2mm_M3, F.Cu at (276.9, 123.2)
- added REF**: MountingHole_3.2mm_M3, Mounting_Holes:MountingHole_3.2mm_M3, F.Cu at (191.0, 96.8)
- added REF**: MountingHole_3.2mm_M3, Mounting_Holes:MountingHole_3.2mm_M3, F.Cu at (33.1, 102.3)
- added REF**: MountingHole_3.2mm_M3, Mounting_Holes:MountingHole_3.2mm_M3, F.Cu at (81.2, 58.9)
- added REF**: MountingHole_3.2mm_M3, Mounting_Holes:MountingHole_3.2mm_M3, F.Cu at (176.3, 59.4)
- added REF**: MountingHole_3.2mm_M3, Mounting_Holes:MountingHole_3.2mm_M3, F.Cu at (242.3, 86.7)
Routing:
- net row4: track 477.3 -> 457.8 mm
- net row0: track 276.5 -> 281.6 mm
- net col9: track 217.2 -> 219.2 mm
- net col4: track 115.8 -> 116.6 mm
- net row1: track 272.7 -> 273.4 mm
Other:
- outline, holes or cut-outs redrawn
